File: hardware/fuse-board/fuse-board.kicad_pcb (KiCad board)
At the start: 2 copper layers, 88 x 76 mm, 43 parts, among them J1 BUS+ IN, J10 W8, J11 SPARE, J12 W21, J13 W22, J14 24V IN, J15 STAR, J16 FRAME, J17 I2C GH, J2 W10, J3 W11, J4 W12, J5 W13, J6 W14, J7 W15, J8 W16, J9 W17, U1 INA228

Commit message: Body B5 for D65 and D66: the fuse board on the 10S bus with the TRACO 12 V rail and the turret's own feed
Holders: F7 the TRACO TEP 150-4812WI's input (W16, 10 A); F8 the turret's feed from the + bus through the stop
relay's pole B (W22, 7.5 A: keeps the G2RL-2's contact under its 8 A carry; its 2-pole DC curve holds about 6 A at
41 V, the turret's 140 W burst is 3.4 A there); F9, F10 spares (no charge port under D65); the 24 V island becomes the
12 V rail (J14 12V IN from the TRACO, W40 14 AWG, 12.5 A at +0.4 C in the pour): F11 the J501 at 12 V (W21, 10 A), F12
the rest of the rail (W43, 7.5 A). Same outline, mounting and copper; DRC, ERC and parity clean; JLCPCB's price
re-read on the new zip: $40.60 for 5. cad/body_fuse_board.py's P3 rows and order follow ($154.48 for one board),
the 7.5 A MINI 58V fuse appended to the catalogue, the doc revised with the relay's rating, the arrival checks and
the plate's third tie slot (40c427b moved it from y 24 to 18, under F12).

Co-Authored-By: Claude Opus 5.5 <noreply@anthropic.com>
Parts:
- F11: value J501 24V 5 A -> J501 12V 10 A
- F12: value TURRET 24V 5 A -> 12V RAIL 7.5 A
- F7: value DDR-120C IN 10 A -> TRACO 12V IN 10 A
- F8: value DDR-60L IN 5 A -> TURRET 7.5 A
- F9: value CHARGE PORT 10 A -> SPARE (no fuse)
- J10: value W8 -> SPARE
- J13: value W22 -> W43
- J14: value 24V IN -> 12V IN
- J9: value W17 -> W22
Connections:
- net +24V renamed +12V
- net OUT_SPARE renamed OUT_SPARE10
- net OUT_W8 renamed OUT_SPARE9
- F12 pad 2: OUT_W22 -> OUT_W43
- F8 pad 2: OUT_W17 -> OUT_W22
- J13 pad 1: OUT_W22 -> OUT_W43
- J9 pad 1: OUT_W17 -> OUT_W22
Routing:
- net OUT_W17: track 19.2 -> 0.00 mm
- net OUT_W43: track 0.00 -> 15.8 mm
- net OUT_W22: track 15.8 -> 19.2 mm
- net +12V: vias 4 -> 6
Other:
- board text added: "12V IN"
- board text added: "PULL A FUSE ONLY WITH BOTH PACKS OUT"
- board text added: "W21 10A"
- board text added: "W22 7.5A"
- board text added: "W43"
- board text added: "W43 7.5A"
- board text removed: "24V IN"
- board text removed: "PULL A FUSE ONLY WITH THE PACK UNPLUGGED"
- board text removed: "W17"
- board text removed: "W17 5A"
- board text removed: "W21 5A"
- board text removed: "W22 5A"
- board text removed: "W8"
- board text removed: "W8 10A"
